File: lab3-new/Assignment Deliverables/pcb/lab3.kicad_pcb (KiCad board)
At the start: 2 copper layers, 32 x 50.8 mm, 15 parts, among them J1 Conn_01x01_Male, J2 USB_A, J3 Conn_01x01_Male, U1 Regulator

Commit message: final project deliverables
Other:
- rule via_min_drill: 0.2 -> 0.3
Changed lines of the file:
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@@
     (via_drill 0.4)
     (via_min_size 0.4)
-    (via_min_drill 0.2)
+    (via_min_drill 0.3)
     (uvia_size 0.3)
     (uvia_drill 0.1)
@@
     (visible_elements 7FFFFFFF)
     (pcbplotparams
-      (layerselection 0x010e8_ffffffff)
+      (layerselection 0x010fc_ffffffff)
       (usegerberextensions false)
       (usegerberattributes false)
@@
       (outputformat 1)
       (mirror false)
-      (drillshape 0)
+      (drillshape 1)
       (scaleselection 1)
-      (outputdirectory "./"))
+      (outputdirectory ""))
   )
   (net 0 "")
