File: microbug/microbug.kicad_pcb (KiCad board)
At the start: 2 copper layers, 31.7 x 38.1 mm, 24 parts, among them J1 Conn_01x03, J2 Conn_01x03, J3 Conn_01x02, M1 Motor_DC, M2 Motor_DC, U1 ATtiny1616-S, U2 QRE1113GR, U3 TC78H651AFNG, U4 QRE1113GR

Commit message: almost done
Parts:
- C2, C3, R6, R7, R8: moved to B.Cu
- moved R2 9.37 mm to (58.9, 70.6), turned to 90 degrees
- moved U4 4.72 mm to (74.9, 67.3), turned to 180 degrees
- moved R5 1.70 mm to (69.6, 64.8)
- moved R4 1.02 mm to (70.6, 60.5), turned to 0 degrees
- moved C3 0.76 mm to (70.9, 69.6), turned to 180 degrees
- moved R6 0.28 mm to (52.6, 65.8)
- moved R3 0.25 mm to (61.0, 64.8)
Routing:
- net GND: track 0.00 -> 104.0 mm, vias 0 -> 3
- net +3V3: track 0.00 -> 77.3 mm, vias 0 -> 2
- net /IR2: track 0.00 -> 52.7 mm
- net /OUT2: track 0.00 -> 50.2 mm, vias 0 -> 2
- net Net-(BT1-Pad1): track 0.00 -> 41.8 mm
- net /OUT1: track 0.00 -> 37.2 mm
- net /LED2: track 0.00 -> 33.8 mm
- net /PWM2: track 0.00 -> 29.9 mm, vias 0 -> 2
- net /UDPI: track 0.00 -> 29.7 mm
- net Net-(M1-Pad2): track 0.00 -> 29.2 mm, vias 0 -> 1
- net /LED3: track 0.00 -> 28.5 mm, vias 0 -> 2
- net /DAC: track 0.00 -> 28.4 mm, vias 0 -> 2
- net /DIR1: track 0.00 -> 26.9 mm
- net /LED1: track 0.00 -> 24.7 mm
- net /PWM1: track 0.00 -> 24.6 mm
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
Commit message: finished
Parts:
- M1, M2: moved to B.Cu
- moved M2 15.8 mm to (56.4, 87.6)
- moved M1 15.5 mm to (71.9, 87.6)
- moved D2 2.96 mm to (65.5, 58.4), turned to 180 degrees
- moved J1 2.79 mm to (64.3, 67.1)
- moved J3 2.03 mm to (63.0, 70.9)
- moved D1 1.61 mm to (77.2, 70.6)
- moved D3 0.25 mm to (51.6, 73.7)
Routing:
- net GND: track 104.0 -> 127.1 mm
- net /DIR2: track 4.43 -> 27.3 mm, vias 1 -> 4
- net Net-(M2-Pad1): track 14.5 -> 31.2 mm, vias 1 -> 2
- net Net-(M2-Pad2): track 13.1 -> 26.4 mm, vias 1 -> 2
- net Net-(M1-Pad2): track 29.2 -> 21.3 mm, vias 1 -> 2
- net Net-(M1-Pad1): track 19.4 -> 12.8 mm, vias 1 -> 2
- net /IR2: track 52.7 -> 58.0 mm
- net /LED2: track 33.8 -> 37.7 mm
- net Net-(D2-Pad2): track 16.2 -> 13.4 mm
- net Net-(BT1-Pad1): track 41.8 -> 44.6 mm
- net Net-(J1-Pad2): track 9.24 -> 11.6 mm
- net +3V3: track 77.3 -> 79.4 mm
- net /DAC: track 28.4 -> 30.3 mm
- net /LED3: track 28.5 -> 26.9 mm
- net /UDPI: track 29.7 -> 31.3 mm
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Other:
- rule trace_min: 0.1524 -> 0.1

Commit message: added logo
Parts:
- added G***: LOGO, microbug-fplib:ieee_logo, F.Cu at (76.7, 92.5)
Other:
- rule trace_min: 0.1 -> 0.1524
- rule via_min_drill: 0.3 -> 0.199898
