File: HOPE_finalProj/HOPE_finalProj.kicad_pcb (KiCad board)
At the start: 2 copper layers, 36 parts, among them M1 Mixer, SW1 SW_Push_DPDT, U1 LM386N-3_NOPB, U2 NE5534, U3 NE5534, U4 LM386N-3_NOPB, Y1 Crystal

Commit message: Layout finished
Parts:
- added BT1: Battery_Cell, digikey-footprints:Battery_Holder_9V_BC9VPC-ND, F.Cu at (150.4, 119.9)
- added C10: 1u, Capacitor_THT:C_Disc_D3.0mm_W1.6mm_P2.50mm, F.Cu at (146.3, 78.7)
- added SW2: SW_SPDT, digikey-footprints:Switch_Slide_11.6x4mm_EG1218, F.Cu at (138.2, 108.5)
- Y1: moved to B.Cu
- moved R8 46.3 mm to (111.8, 66.8)
- moved AE1 43.3 mm to (133.6, 60.5), turned to 0 degrees
- moved C9 43.1 mm to (113.8, 63.5)
- moved Y1 37.3 mm to (159.8, 92.5), turned to 180 degrees
- moved LS1 36.9 mm to (147.8, 93.5), turned to 0 degrees
- moved R10 32.2 mm to (153.7, 109.7), turned to 180 degrees
- moved R3 27.4 mm to (147.8, 64.5), turned to 180 degrees
- moved MK1 24.9 mm to (132.6, 86.6)
- moved C3 24.7 mm to (129.0, 78.0)
- moved C1 24.3 mm to (128.8, 68.6)
- moved R11 23.6 mm to (147.8, 72.6), turned to 180 degrees
- moved R7 23.0 mm to (110.0, 89.7)
- moved R12 22.6 mm to (166.1, 77.2), turned to 90 degrees
- moved R2 21.6 mm to (147.8, 68.6)
- moved R1 20.3 mm to (129.0, 72.4), turned to 0 degrees
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Connections:
- AE1 pad 1: Net-(AE1-Pad1) -> /ANT
- C12 pad 2: Net-(AE1-Pad1) -> /ANT
- C13 pad 2: Net-(C13-Pad2) -> Net-(C10-Pad2)
- C14 pad 2: Net-(C13-Pad2) -> Net-(C10-Pad2)
- C6 pad 1: Net-(C6-Pad1) -> /ANT
- LS1 pad 1: Net-(C13-Pad2) -> Net-(C10-Pad1)
- R12 pad 2: Net-(AE1-Pad1) -> /ANT
- R13 pad 2: Net-(C13-Pad2) -> Net-(C10-Pad2)
- R7 pad 1: Net-(C6-Pad1) -> /ANT
- U2 pad 2: Net-(C6-Pad1) -> /ANT
- U3 pad 6: Net-(AE1-Pad1) -> /ANT
- U4 pad 5: Net-(C13-Pad2) -> Net-(C10-Pad2)
Routing:
- net /ANT: track 0.00 -> 112.4 mm
- net Net-(C13-Pad2): track 54.2 -> 0.00 mm
- net Net-(C10-Pad2): track 0.00 -> 42.6 mm
- net Net-(C9-Pad1): track 23.5 -> 65.9 mm
- net Net-(AE1-Pad1): track 33.4 -> 0.00 mm
- net Net-(C2-Pad1): track 24.3 -> 55.1 mm
- net Net-(C6-Pad1): track 28.4 -> 0.00 mm
- net GND: track 161.0 -> 182.1 mm
- net Net-(C13-Pad1): track 59.7 -> 39.5 mm
- net Net-(C10-Pad1): track 0.00 -> 16.1 mm
- net Net-(M1-Pad1): track 29.6 -> 40.9 mm
- net Net-(C7-Pad2): track 19.4 -> 8.78 mm
- net Net-(M1-Pad2): track 25.6 -> 35.0 mm
- net Net-(C12-Pad1): track 35.5 -> 41.9 mm
- net Net-(C8-Pad2): track 9.93 -> 15.0 mm
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Other:
- board outline added: 69.3 x 95 mm

Commit message: Fixed battery
Parts:
- removed BT1: Battery_Cell, digikey-footprints:Battery_Holder_9V_BC9VPC-ND
- added BAT1: BC9VPC, digikey-footprints:Battery_Holder_9V_BC9VPC-ND, F.Cu at (149.9, 118.9)
Connections:
- SW2 pad 1: (no net) -> Net-(BAT1-PadNEG)
Routing:
- net Net-(BAT1-PadNEG): track 0.00 -> 38.2 mm
- net VCC: track 135.3 -> 151.7 mm
Changed lines of the file:
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@@
     (thickness 1.6)
     (drawings 4)
-    (tracks 272)
+    (tracks 276)
     (zones 0)
     (modules 39)
-    (nets 22)
+    (nets 23)
   )
   (page A4)
@@
   (net 20 "Net-(C10-Pad2)")
   (net 21 "Net-(C10-Pad1)")
+  (net 22 "Net-(BAT1-PadNEG)")
   (net_class Default "This is the default net class."
     (clearance 0.2)
@@
     (add_net /ANT)
     (add_net GND)
+    (add_net "Net-(BAT1-PadNEG)")
     (add_net "Net-(C1-Pad1)")
     (add_net "Net-(C1-Pad2)")
@@
     (add_net "Net-(M1-Pad6)")
     (add_net "Net-(M1-Pad7)")
+    (add_net "Net-(M1-Pad8)")
+    (add_net "Net-(SW1-Pad1)")
+    (add_net "Net-(SW1-Pad6)")
+    (add_net "Net-(SW2-Pad3)")
+    (add_net "Net-(U1-Pad1)")
+    (add_net "Net-(U1-Pad7)")
+    (add_net "Net-(U1-Pad8)")
+    (add_net "Net-(U2-Pad1)")
+    (add_net "Net-(U2-Pad4)")
+    (add_net "Net-(U2-Pad5)")
+    (add_net "Net-(U2-Pad7)")
+    (add_net "Net-(U2-Pad8)")
+    (add_net "Net-(U3-Pad1)")
+    (add_net "Net-(U3-Pad4)")
+    (add_net "Net-(U3-Pad5)")
+    (add_net "Net-(U3-Pad7)")
+    (add_net "Net-(U3-Pad8)")
+    (add_net "Net-(U4-Pad1)")
+    (add_net "Net-(U4-Pad7)")
+    (add_net "Net-(U4-Pad8)")
     (add_net VCC)
   )
   (module digikey-footprints:Battery_Holder_9V_BC9VPC-ND (layer F.Cu)
-    (at 150.368 119.888)
+    (at 149.86 118.872)
     (descr http://www.memoryprotectiondevices.com/datasheets/BC9VPC-datasheet.pdf)
-    (fp_text reference BT1 (at -12.54 -4.91) (layer F.SilkS)
-      (effects (font (size 1 1) (thickness 0.15)))
-    )
-    (fp_text value Battery_Cell (at -12.01 27.63) (layer F.Fab)
+    (fp_text reference BAT1 (at -12.54 -4.91) (layer F.SilkS)
+      (effects (font (size 1 1) (thickness 0.15)))
+    )
+    (fp_text value BC9VPC (at -12.01 27.63) (layer F.Fab)
       (effects (font (size 1 1) (thickness 0.15)))
     )
@@
       (effects (font (size 1 1) (thickness 0.15)))
     )
-    (pad POS thru_hole oval (at 12.62 4.74) (size 1.75 3.3) (drill oval 0.75 2.3) (layers *.Cu *.Mask))
+    (pad POS thru_hole circle (at 12.62 4.74 180) (size 1.75 1.75) (drill 0.75) (layers *.Cu *.Mask)
+      (net 6 VCC))
     (pad "" np_thru_hole circle (at -26.87 0) (size 5.57 5.57) (drill 5.57) (layers *.Cu *.Mask))
     (pad "" np_thru_hole circle (at 0 0) (size 5.57 5.57) (drill 5.57) (layers *.Cu *.Mask))
     (pad "" np_thru_hole circle (at -13.49 22.5) (size 5.57 5.57) (drill 5.57) (layers *.Cu *.Mask))
-    (pad NEG thru_hole oval (at 12.62 17.69) (size 1.75 3.3) (drill oval 0.75 2.3) (layers *.Cu *.Mask))
+    (pad NEG thru_hole circle (at 12.62 17.69) (size 1.75 1.75) (drill 0.75) (layers *.Cu *.Mask)
+      (net 22 "Net-(BAT1-PadNEG)"))
   )
   (module HOPE_finalProj_lib:Crystal (layer B.Cu)
@@
     (pad 2 thru_hole circle (at 2.5 0 180) (size 1.9 1.9) (drill 0.9) (layers *.Cu *.Mask)
       (net 3 GND))
-    (pad 1 thru_hole rect (at 0 0 180) (size 1.9 1.9) (drill 0.9) (layers *.Cu *.Mask))
+    (pad 1 thru_hole rect (at 0 0 180) (size 1.9 1.9) (drill 0.9) (layers *.Cu *.Mask)
+      (net 22 "Net-(BAT1-PadNEG)"))
   )
   (module Capacitor_THT:C_Disc_D3.0mm_W1.6mm_P2.50mm (layer F.Cu)
@@
   (segment (start 137.670001 100.367999) (end 132.879999 100.367999) (width 0.25) (layer F.Cu) (net 6))
   (segment (start 138.47 99.568) (end 137.670001 100.367999) (width 0.25) (layer F.Cu) (net 6))
+  (segment (start 156.464 117.596) (end 162.48 123.612) (width 0.25) (layer B.Cu) (net 6))
+  (segment (start 156.464 109.728) (end 156.464 117.596) (width 0.25) (layer B.Cu) (net 6))
   (segment (start 109.982 110.744) (end 109.982 106.934) (width 0.25) (layer F.Cu) (net 7))
   (segment (start 113.792 100.584) (end 114.808 99.568) (width 0.25) (layer F.Cu) (net 7))
@@
   (segment (start 146.304 93.19749) (end 146.57851 93.472) (width 0.25) (layer F.Cu) (net 21))
   (segment (start 146.304 78.7) (end 146.304 93.19749) (width 0.25) (layer F.Cu) (net 21))
+  (segment (start 138.176 112.258) (end 162.48 136.562) (width 0.25) (layer B.Cu) (net 22))
+  (segment (start 138.176 108.458) (end 138.176 112.258) (width 0.25) (layer B.Cu) (net 22))
 )

Commit message: Doing layout
Parts:
- removed SW2: SW_SPDT, digikey-footprints:Switch_Slide_11.6x4mm_EG1218
- added C15: 1u, Capacitor_THT:C_Disc_D3.0mm_W1.6mm_P2.50mm, F.Cu at (121.2, 114.5)
- added C16: 1u, Capacitor_THT:C_Disc_D3.0mm_W1.6mm_P2.50mm, F.Cu at (126.9, 114.5)
- added C17: 1u, Capacitor_THT:C_Disc_D3.0mm_W1.6mm_P2.50mm, F.Cu at (132.5, 114.5)
- added C18: 1u, Capacitor_THT:C_Disc_D3.0mm_W1.6mm_P2.50mm, F.Cu at (138.2, 114.5)
- added SW3: SW_Push_DPDT, HOPE_finalProj_lib:DPDT_Switch, F.Cu at (136.6, 108.2)
- moved BAT1 5.18 mm to (150.9, 124.0)
- moved SW1 4.85 mm to (128.0, 95.8), turned to 0 degrees
Connections:
- BAT1 pad NEG: Net-(BAT1-PadNEG) -> GND
- C14 pad 1: VCC -> speaker_VCC
- M1 pad 8: (no net) -> VCC
- SW1 pad 1: (no net) -> Net-(C15-Pad1)
- SW1 pad 2: Net-(C7-Pad2) -> Net-(M1-Pad1)
- SW1 pad 3: Net-(M1-Pad1) -> Net-(C7-Pad2)
- SW1 pad 4: Net-(M1-Pad2) -> Net-(C8-Pad2)
- SW1 pad 5: Net-(C8-Pad2) -> Net-(M1-Pad2)
- SW1 pad 6: (no net) -> Net-(C16-Pad2)
- U1 pad 1: (no net) -> Net-(U1-Pad1)
- U1 pad 7: (no net) -> Net-(U1-Pad7)
- U1 pad 8: (no net) -> Net-(U1-Pad8)
- U2 pad 1: (no net) -> Net-(U2-Pad1)
- U2 pad 4: (no net) -> GND
- U2 pad 5: (no net) -> Net-(U2-Pad5)
- U2 pad 7: (no net) -> VCC
- U2 pad 8: (no net) -> Net-(U2-Pad8)
- U3 pad 1: (no net) -> Net-(U3-Pad1)
- U3 pad 4: (no net) -> GND
- U3 pad 5: (no net) -> Net-(U3-Pad5)
- U3 pad 7: (no net) -> transmitter_VCC
- U3 pad 8: (no net) -> Net-(U3-Pad8)
- U4 pad 1: (no net) -> Net-(U4-Pad1)
- U4 pad 6: VCC -> speaker_VCC
- U4 pad 7: (no net) -> Net-(U4-Pad7)
- U4 pad 8: (no net) -> Net-(U4-Pad8)
Routing:
- net Net-(M1-Pad1): track 40.9 -> 0.00 mm
- net Net-(BAT1-PadNEG): track 38.2 -> 0.00 mm
- net GND: track 182.1 -> 146.9 mm
- net Net-(M1-Pad2): track 35.0 -> 0.00 mm
- net VCC: track 151.7 -> 135.3 mm
- net Net-(C8-Pad2): track 15.0 -> 0.00 mm
- net Net-(C7-Pad2): track 8.78 -> 0.00 mm

Commit message: Finished layout
Parts:
- BAT1: moved to B.Cu
- moved BAT1 22.6 mm to (151.1, 146.6)
- moved SW3 9.54 mm to (128.0, 104.1)
- moved R10 7.37 mm to (146.3, 109.7), turned to 0 degrees
- moved C8 7.17 mm to (123.2, 110.0), turned to 0 degrees
- moved C18 2.55 mm to (140.7, 114.5), turned to 180 degrees
- moved C15 2.48 mm to (123.7, 114.5), turned to 180 degrees
Routing:
- net GND: track 146.9 -> 238.7 mm
- net transmitter_VCC: track 0.00 -> 85.8 mm, vias 0 -> 1
- net VCC: track 135.3 -> 202.5 mm, vias 0 -> 1
- net Net-(M1-Pad2): track 0.00 -> 59.1 mm
- net speaker_VCC: track 0.00 -> 48.5 mm
- net Net-(M1-Pad1): track 0.00 -> 47.7 mm
- net Net-(C15-Pad1): track 0.00 -> 30.4 mm
- net Net-(C17-Pad2): track 0.00 -> 17.8 mm, vias 0 -> 1
- net Net-(C16-Pad2): track 0.00 -> 16.8 mm
- net Net-(C18-Pad2): track 0.00 -> 13.6 mm
- net Net-(C8-Pad2): track 0.00 -> 12.5 mm
- net Net-(C7-Pad2): track 0.00 -> 8.64 mm
- net Net-(C6-Pad2): track 29.4 -> 36.0 mm
- net Net-(C11-Pad1): track 56.7 -> 59.6 mm
Other:
- board size 69.3 x 95 mm -> 62 x 95 mm

Commit message: fixed unconnected components
Routing:
- net GND: track 238.7 -> 244.0 mm
Changed lines of the file:
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@@
-(kicad_pcb (version 20171130) (host pcbnew "(5.1.5-0-10_14)")
+(kicad_pcb (version 20171130) (host pcbnew "(5.1.5)-3")
   (general
     (thickness 1.6)
     (drawings 4)
-    (tracks 376)
+    (tracks 378)
     (zones 0)
     (modules 43)
@@
     (solder_mask_min_width 0.25)
     (aux_axis_origin 0 0)
-    (visible_elements FFFFFF7F)
+    (visible_elements 7FFFFFFF)
     (pcbplotparams
       (layerselection 0x010fc_ffffffff)
@@
       (outputformat 1)
       (mirror false)
-      (drillshape 1)
+      (drillshape 0)
       (scaleselection 1)
       (outputdirectory ""))
@@
   (segment (start 163.75 115.236) (end 163.75 128.868) (width 0.25) (layer F.Cu) (net 3))
   (segment (start 163.041 114.527) (end 163.75 115.236) (width 0.25) (layer F.Cu) (net 3))
+  (segment (start 110.958 102.108) (end 109.982 103.084) (width 0.25) (layer F.Cu) (net 3))
+  (segment (start 114.808 102.108) (end 110.958 102.108) (width 0.25) (layer F.Cu) (net 3))
   (segment (start 111.76 75.184) (end 110.49 73.914) (width 0.25) (layer B.Cu) (net 4))
   (segment (start 133.566001 67.780001) (end 134.366 68.58) (width 0.25) (layer B.Cu) (net 4))
