File: HOPE_finalProj/HOPE_finalProj.kicad_pcb (KiCad board)
At the start: 2 copper layers, 62 x 95 mm, 43 parts, among them M1 Mixer, SW1 SW_Push_DPDT, SW3 SW_Push_DPDT, U1 LM386N-3_NOPB, U2 NE5534, U3 NE5534, U4 LM386N-3_NOPB, Y1 Crystal

Commit message: Change 10pF capacitors: cheaper and smaller
Parts:
- C12, C13, C3, C6: footprint Capacitor_THT:C_Disc_D7.5mm_W5.0mm_P7.50mm -> Capacitor_THT:C_Disc_D5.0mm_W2.5mm_P2.50mm
Routing:
- net /ANT: track 112.4 -> 107.2 mm
- net Net-(C6-Pad2): track 36.0 -> 41.0 mm
- net Net-(C10-Pad2): track 42.6 -> 47.6 mm
- net Net-(C3-Pad2): track 64.2 -> 64.0 mm, vias 0 -> 1
